File: Phase B/PCB_Projects/2025_04_STM32F103_RobotBrain /2025_04_STM32F103_RobotBrain.kicad_sch (KiCad schematic)
At the start: 47 parts, among them J1 USB_B_Mini, J10 CONN_TRACK, J11 CONN_UART, J2 CONN_MPU6050, J3 CONN_ULTRA, J4 CONN_SWD, J5 CONN_5V, J6 CONN_3V3, J7 CONN_DRIVE, J8 CONN_HAL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

Commit message: Robot Brain project, reformat repo
Other:
- company: Goncalo Martins -> Winston Har
Changed lines of the file:
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@@
 	(title_block
 		(title "Robot Brain PCB Board")
-		(date "2025-04-30")
+		(date "2025-05-06")
 		(rev "1.0")
-		(company "Goncalo Martins")
+		(company "Winston Har")
 	)
 	(rectangle
